File: KiCad/proj_seients/proj_seients.kicad_sch (KiCad schematic)
At the start: 0 parts

Commit message: Versió 1.0 Layout
Changed lines of the file:
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@@
 	(text "Pàgina principal"
 		(exclude_from_sim no)
-		(at 191.008 172.72 0)
+		(at 190.754 179.07 0)
 		(effects
 			(font
@@
 	(text "Autors: Miguel Tovar i Pol Salas"
 		(exclude_from_sim no)
-		(at 203.708 168.91 0)
+		(at 203.454 175.26 0)
 		(effects
 			(font
