File: KiCad/proj_seients/potencia.kicad_sch (KiCad schematic)
At the start: 35 parts, among them J1 BATERIA 12V, J19 J_SENSOR_TEMP, J4 Motor, J5 Motor, J6 Motor, J7 Manta_Asiento, Q1 IRLZ44N, U2 LM2596S-5, U3 LM1117DT-3.3, U5 PCA9685BS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

Commit message: V3.6
Connections:
- net at U7.6 (OUT1): now also J4.1 (Pin_1); no longer J4.2 (Pin_2)
- net at U7.8 (OUT2): now also J4.2 (Pin_2); no longer J4.1 (Pin_1)
- net at U8.6 (OUT1): now also J5.1 (Pin_1); no longer J5.2 (Pin_2)
- net at U8.8 (OUT2): now also J5.2 (Pin_2); no longer J5.1 (Pin_1)
- net at J6.1 (Pin_1): now also U6.6 (OUT1); no longer U6.8 (OUT2)
- net at J6.2 (Pin_2): now also U6.8 (OUT2); no longer U6.6 (OUT1)
Changed lines of the file:
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@@
 	(symbol
 		(lib_id "Connector:Screw_Terminal_01x02")
-		(at 182.88 121.92 0)
-		(mirror x)
+		(at 182.88 119.38 0)
 		(unit 1)
 		(exclude_from_sim no)
@@
 		(dnp no)
 		(property "Reference" "J6"
-			(at 182.88 115.316 0)
+			(at 182.88 125.984 0)
 			(effects
 				(font
@@
 		)
 		(property "Value" "Motor"
-			(at 183.388 117.094 0)
+			(at 183.388 124.206 0)
 			(effects
 				(font
@@
 		)
 		(property "Footprint" "TerminalBlock_Phoenix:TerminalBlock_Phoenix_MKDS-1,5-2-5.08_1x02_P5.08mm_Horizontal"
-			(at 182.88 121.92 0)
+			(at 182.88 119.38 0)
 			(effects
 				(font
@@
 		)
 		(property "Datasheet" "~"
-			(at 182.88 121.92 0)
+			(at 182.88 119.38 0)
 			(effects
 				(font
@@
 		)
 		(property "Description" "Generic screw terminal, single row, 01x02, script generated (kicad-library-utils/schlib/autogen/connector/)"
-			(at 182.88 121.92 0)
+			(at 182.88 119.38 0)
 			(effects
 				(font
@@
 	(symbol
 		(lib_id "Connector:Screw_Terminal_01x02")
-		(at 182.88 86.36 0)
-		(mirror x)
+		(at 182.88 83.82 0)
 		(unit 1)
 		(exclude_from_sim no)
@@
 		(dnp no)
 		(property "Reference" "J5"
-			(at 182.88 79.756 0)
+			(at 182.88 90.424 0)
 			(effects
 				(font
@@
 		)
 		(property "Value" "Motor"
-			(at 183.388 81.534 0)
+			(at 183.388 88.646 0)
 			(effects
 				(font
@@
 		)
 		(property "Footprint" "TerminalBlock_Phoenix:TerminalBlock_Phoenix_MKDS-1,5-2-5.08_1x02_P5.08mm_Horizontal"
-			(at 182.88 86.36 0)
+			(at 182.88 83.82 0)
 			(effects
 				(font
@@
 		)
 		(property "Datasheet" "~"
-			(at 182.88 86.36 0)
+			(at 182.88 83.82 0)
 			(effects
 				(font
@@
 		)
 		(property "Description" "Generic screw terminal, single row, 01x02, script generated (kicad-library-utils/schlib/autogen/connector/)"
-			(at 182.88 86.36 0)
+			(at 182.88 83.82 0)
 			(effects
 				(font
@@
 	(symbol
 		(lib_id "Connector:Screw_Terminal_01x02")
-		(at 182.88 49.53 0)
-		(mirror x)
+		(at 182.88 46.99 0)
 		(unit 1)
 		(exclude_from_sim no)
@@
 		(dnp no)
 		(property "Reference" "J4"
-			(at 182.88 42.926 0)
+			(at 182.88 53.594 0)
 			(effects
 				(font
@@
 		)
 		(property "Value" "Motor"
-			(at 183.388 44.704 0)
+			(at 183.388 51.816 0)
 			(effects
 				(font
@@
 		)
 		(property "Footprint" "TerminalBlock_Phoenix:TerminalBlock_Phoenix_MKDS-1,5-2-5.08_1x02_P5.08mm_Horizontal"
-			(at 182.88 49.53 0)
+			(at 182.88 46.99 0)
 			(effects
 				(font
@@
 		)
 		(property "Datasheet" "~"
-			(at 182.88 49.53 0)
+			(at 182.88 46.99 0)
 			(effects
 				(font
@@
 		)
 		(property "Description" "Generic screw terminal, single row, 01x02, script generated (kicad-library-utils/schlib/autogen/connector/)"
-			(at 182.88 49.53 0)
-			(effects
-				(font
+			(at 182.88 46.99 0)
+			(effects
+				(font
