File: KiCad/proj_seients/potencia.kicad_sch (KiCad schematic)
At the start: 35 parts, among them J1 BATERIA 12V, J19 J_SENSOR_TEMP, J4 Motor, J5 Motor, J6 Motor, J7 Manta_Asiento, Q1 IRLZ44N, U2 LM2596S-5, U3 LM1117DT-3.3, U5 PCA9685BS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

Commit message: V3.2
Connections:
- net 12V: now also J7.1 (Pin_1); no longer J7.2 (Pin_2)
- net GND: now also J1.2 (Pin_2); no longer J1.1 (Pin_1)
- net at Q1.2 (D): now also J7.2 (Pin_2); no longer J7.1 (Pin_1)
- net at D1.2 (A): now also J1.1 (Pin_1); no longer J1.2 (Pin_2)
Other:
- moved on the sheet: J1, J19, J7, R3
Changed lines of the file:
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@@
 	)
 	(junction
-		(at 44.45 132.08)
+		(at 44.45 134.62)
 		(diameter 0)
 		(color 0 0 0 0)
@@
 	)
 	(junction
-		(at 46.99 123.19)
+		(at 46.99 125.73)
 		(diameter 0)
 		(color 0 0 0 0)
@@
 	(wire
 		(pts
-			(xy 50.8 128.27) (xy 46.99 128.27)
+			(xy 50.8 125.73) (xy 46.99 125.73)
 		)
 		(stroke
@@
 	(wire
 		(pts
-			(xy 58.42 123.19) (xy 57.15 123.19)
+			(xy 46.99 115.57) (xy 46.99 116.84)
 		)
 		(stroke
@@
 	(wire
 		(pts
-			(xy 44.45 123.19) (xy 46.99 123.19)
+			(xy 44.45 125.73) (xy 46.99 125.73)
 		)
 		(stroke
@@
 	(wire
 		(pts
-			(xy 46.99 128.27) (xy 46.99 123.19)
-		)
-		(stroke
-			(width 0)
-			(type default)
-		)
-	)
-	(wire
-		(pts
 			(xy 200.66 62.23) (xy 200.66 63.5)
 		)
@@
 	(wire
 		(pts
-			(xy 44.45 125.73) (xy 44.45 132.08)
-		)
-		(stroke
-			(width 0)
-			(type default)
-		)
-	)
-	(wire
-		(pts
-			(xy 46.99 123.19) (xy 49.53 123.19)
+			(xy 44.45 128.27) (xy 44.45 134.62)
 		)
 		(stroke
@@
 	(wire
 		(pts
+			(xy 46.99 124.46) (xy 46.99 125.73)
+		)
+		(stroke
+			(width 0)
+			(type default)
+		)
+	)
+	(wire
+		(pts
 			(xy 175.26 83.82) (xy 177.8 83.82)
 		)
@@
 	(global_label "TEMP_SEIENT"
 		(shape output)
-		(at 50.8 128.27 0)
+		(at 50.8 125.73 0)
 		(fields_autoplaced yes)
 		(effects
@@
 		)
 		(property "Intersheetrefs" "${INTERSHEET_REFS}"
-			(at 66.0012 128.27 0)
+			(at 66.0012 125.73 0)
 			(effects
 				(font
@@
 	(global_label "3.3V"
 		(shape input)
-		(at 58.42 123.19 0)
+		(at 46.99 115.57 90)
 		(fields_autoplaced yes)
 		(effects
@@
 		)
 		(property "Intersheetrefs" "${INTERSHEET_REFS}"
-			(at 65.5176 123.19 0)
+			(at 46.99 108.4724 90)
 			(effects
 				(font
@@
 	(symbol
 		(lib_id "Device:R")
-		(at 53.34 123.19 90)
+		(at 46.99 120.65 180)
 		(unit 1)
 		(exclude_from_sim no)
@@
 		(dnp no)
 		(property "Reference" "R3"
-			(at 51.816 125.222 90)
+			(at 49.022 122.174 90)
 			(effects
 				(font
@@
 		)
 		(property "Value" "10k"
-			(at 55.88 125.222 90)
+			(at 49.022 118.11 90)
 			(effects
 				(font
@@
 		)
 		(property "Footprint" "Resistor_SMD:R_0805_2012Metric"
-			(at 53.34 124.968 90)
+			(at 48.768 120.65 90)
 			(effects
 				(font
@@
 		)
 		(property "Datasheet" "~"
-			(at 53.34 123.19 0)
+			(at 46.99 120.65 0)
 			(effects
 				(font
@@
 		)
 		(property "Description" "Resistor"
-			(at 53.34 123.19 0)
+			(at 46.99 120.65 0)
 			(effects
 				(font
@@
 	(symbol
 		(lib_id "power:PWR_FLAG")
-		(at 44.45 132.08 90)
+		(at 44.45 134.62 90)
 		(unit 1)
 		(exclude_from_sim no)
@@
 		(dnp no)
 		(property "Reference" "#FLG05"
-			(at 42.545 132.08 0)
+			(at 42.545 134.62 0)
 			(effects
 				(font
@@
 		)
 		(property "Value" "PWR_FLAG"
-			(at 43.942 130.048 90)
+			(at 43.942 132.588 90)
 			(effects
 				(font
@@
 		)
 		(property "Footprint" ""
-			(at 44.45 132.08 0)
+			(at 44.45 134.62 0)
 			(effects
 				(font
@@
 		)
 		(property "Datasheet" "~"
-			(at 44.45 132.08 0)
+			(at 44.45 134.62 0)
 			(effects
 				(font
@@
 		)
 		(property "Description" "Special symbol for telling ERC where power comes from"
-			(at 44.45 132.08 0)
+			(at 44.45 134.62 0)
 			(effects
 				(font
@@
 	(symbol
 		(lib_id "Connector:Screw_Terminal_01x02")
-		(at 39.37 125.73 180)
+		(at 39.37 128.27 180)
 		(unit 1)
 		(exclude_from_sim no)
@@
 		(dnp no)
 		(property "Reference" "J19"
-			(at 39.37 118.11 0)
+			(at 39.37 120.65 0)
 			(effects
 				(font
@@
 		)
 		(property "Value" "J_SENSOR_TEMP"
-			(at 45.212 120.396 0)
+			(at 36.576 122.428 90)
 			(effects
 				(font
@@
 		)
 		(property "Footprint" "TerminalBlock_Phoenix:TerminalBlock_Phoenix_MKDS-1,5-2-5.08_1x02_P5.08mm_Horizontal"
-			(at 39.37 125.73 0)
+			(at 39.37 128.27 0)
 			(effects
 				(font
@@
 		)
 		(property "Datasheet" "~"
-			(at 39.37 125.73 0)
+			(at 39.37 128.27 0)
 			(effects
 				(font
@@
 		)
 		(property "Description" "Generic screw terminal, single row, 01x02, script generated (kicad-library-utils/schlib/autogen/connector/)"
-			(at 39.37 125.73 0)
+			(at 39.37 128.27 0)
 			(effects
 				(font
@@
 	(symbol
 		(lib_id "power:GND")
-		(at 44.45 132.08 0)
+		(at 44.45 134.62 0)
 		(unit 1)
 		(exclude_from_sim no)
@@
 		(fields_autoplaced yes)
 		(property "Reference" "#PWR0101"
-			(at 44.45 138.43 0)
+			(at 44.45 140.97 0)
 			(effects
 				(font
@@
 		)
 		(property "Value" "GND"
-			(at 44.45 137.16 0)
+			(at 44.45 139.7 0)
 			(effects
 				(font
@@
 		)
 		(property "Footprint" ""
-			(at 44.45 132.08 0)
+			(at 44.45 134.62 0)
 			(effects
 				(font
@@
 		)
 		(property "Datasheet" ""
-			(at 44.45 132.08 0)
+			(at 44.45 134.62 0)
 			(effects
 				(font
@@
 		)
 		(property "Description" "Power symbol creates a global label with name \"GND\" , ground"
-			(at 44.45 132.08 0)
+			(at 44.45 134.62 0)
 			(effects
 				(font
@@
 	(symbol
 		(lib_id "Connector:Screw_Terminal_01x02")
-		(at 40.64 46.99 180)
+		(at 40.64 44.45 0)
+		(mirror y)
 		(unit 1)
 		(exclude_from_sim no)
@@
 		(dnp no)
 		(property "Reference" "J1"
-			(at 40.64 41.402 0)
+			(at 40.64 50.038 0)
 			(effects
 				(font
@@
 		)
 		(property "Value" "BATERIA 12V"
-			(at 37.592 45.974 90)
+			(at 37.592 45.466 90)
 			(effects
 				(font
@@
 		)
 		(property "Footprint" "TerminalBlock_Phoenix:TerminalBlock_Phoenix_MKDS-1,5-2-5.08_1x02_P5.08mm_Horizontal"
-			(at 40.64 46.99 0)
+			(at 40.64 44.45 0)
 			(effects
 				(font
@@
 		)
 		(property "Datasheet" "~"
-			(at 40.64 46.99 0)
+			(at 40.64 44.45 0)
 			(effects
 				(font
@@
 		)
 		(property "Description" "Generic screw terminal, single row, 01x02, script generated (kicad-library-utils/schlib/autogen/connector/)"
-			(at 40.64 46.99 0)
+			(at 40.64 44.45 0)
 			(effects
 				(font
@@
 	(symbol
 		(lib_id "Connector:Screw_Terminal_01x02")
-		(at 78.74 119.38 180)
+		(at 78.74 116.84 0)
+		(mirror y)
 		(unit 1)
 		(exclude_from_sim no)
@@
 		(dnp no)
 		(property "Reference" "J7"
-			(at 75.692 119.38 0)
+			(at 75.692 116.84 0)
 			(effects
 				(font
@@
 		)
 		(property "Value" "Manta_Asiento"
-			(at 76.962 122.174 0)
+			(at 76.962 114.046 0)
 			(effects
 				(font
@@
 		)
 		(property "Footprint" "TerminalBlock_Phoenix:TerminalBlock_Phoenix_MKDS-1,5-2-5.08_1x02_P5.08mm_Horizontal"
-			(at 78.74 119.38 0)
+			(at 78.74 116.84 0)
 			(effects
 				(font
@@
 		)
 		(property "Datasheet" "~"
-			(at 78.74 119.38 0)
+			(at 78.74 116.84 0)
 			(effects
 				(font
@@
 		)
 		(property "Description" "Generic screw terminal, single row, 01x02, script generated (kicad-library-utils/schlib/autogen/connector/)"
-			(at 78.74 119.38 0)
+			(at 78.74 116.84 0)
 			(effects
 				(font

Commit message: V3.7
Connections:
- net GND: now also J1.1 (Pin_1); no longer J1.2 (Pin_2)
- net at U7.6 (OUT1): now also J4.1 (Pin_1); no longer J4.2 (Pin_2)
- net at U7.8 (OUT2): now also J4.2 (Pin_2); no longer J4.1 (Pin_1)
- net at U8.6 (OUT1): now also J5.1 (Pin_1); no longer J5.2 (Pin_2)
- net at U8.8 (OUT2): now also J5.2 (Pin_2); no longer J5.1 (Pin_1)
- net at J6.1 (Pin_1): now also U6.6 (OUT1); no longer U6.8 (OUT2)
- net at J6.2 (Pin_2): now also U6.8 (OUT2); no longer U6.6 (OUT1)
- net at D1.2 (A): now also J1.2 (Pin_2); no longer J1.1 (Pin_1)
Other:
- moved on the sheet: J1
Changed lines of the file:
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@@
 	(symbol
 		(lib_id "Connector:Screw_Terminal_01x02")
-		(at 182.88 121.92 0)
-		(mirror x)
+		(at 182.88 119.38 0)
 		(unit 1)
 		(exclude_from_sim no)
@@
 		(dnp no)
 		(property "Reference" "J6"
-			(at 182.88 115.316 0)
+			(at 182.88 125.984 0)
 			(effects
 				(font
@@
 		)
 		(property "Value" "Motor"
-			(at 183.388 117.094 0)
+			(at 183.388 124.206 0)
 			(effects
 				(font
@@
 		)
 		(property "Footprint" "TerminalBlock_Phoenix:TerminalBlock_Phoenix_MKDS-1,5-2-5.08_1x02_P5.08mm_Horizontal"
-			(at 182.88 121.92 0)
+			(at 182.88 119.38 0)
 			(effects
 				(font
@@
 		)
 		(property "Datasheet" "~"
-			(at 182.88 121.92 0)
+			(at 182.88 119.38 0)
 			(effects
 				(font
@@
 		)
 		(property "Description" "Generic screw terminal, single row, 01x02, script generated (kicad-library-utils/schlib/autogen/connector/)"
-			(at 182.88 121.92 0)
+			(at 182.88 119.38 0)
 			(effects
 				(font
@@
 	(symbol
 		(lib_id "Connector:Screw_Terminal_01x02")
-		(at 182.88 86.36 0)
-		(mirror x)
+		(at 182.88 83.82 0)
 		(unit 1)
 		(exclude_from_sim no)
@@
 		(dnp no)
 		(property "Reference" "J5"
-			(at 182.88 79.756 0)
+			(at 182.88 90.424 0)
 			(effects
 				(font
@@
 		)
 		(property "Value" "Motor"
-			(at 183.388 81.534 0)
+			(at 183.388 88.646 0)
 			(effects
 				(font
@@
 		)
 		(property "Footprint" "TerminalBlock_Phoenix:TerminalBlock_Phoenix_MKDS-1,5-2-5.08_1x02_P5.08mm_Horizontal"
-			(at 182.88 86.36 0)
+			(at 182.88 83.82 0)
 			(effects
 				(font
@@
 		)
 		(property "Datasheet" "~"
-			(at 182.88 86.36 0)
+			(at 182.88 83.82 0)
 			(effects
 				(font
@@
 		)
 		(property "Description" "Generic screw terminal, single row, 01x02, script generated (kicad-library-utils/schlib/autogen/connector/)"
-			(at 182.88 86.36 0)
+			(at 182.88 83.82 0)
 			(effects
 				(font
@@
 	(symbol
 		(lib_id "Connector:Screw_Terminal_01x02")
-		(at 40.64 44.45 0)
-		(mirror y)
+		(at 40.64 46.99 180)
 		(unit 1)
 		(exclude_from_sim no)
@@
 		(dnp no)
 		(property "Reference" "J1"
-			(at 40.64 50.038 0)
+			(at 40.64 41.402 0)
 			(effects
 				(font
@@
 		)
 		(property "Value" "BATERIA 12V"
-			(at 37.592 45.466 90)
+			(at 37.592 45.974 90)
 			(effects
 				(font
@@
 		)
 		(property "Footprint" "TerminalBlock_Phoenix:TerminalBlock_Phoenix_MKDS-1,5-2-5.08_1x02_P5.08mm_Horizontal"
-			(at 40.64 44.45 0)
+			(at 40.64 46.99 0)
 			(effects
 				(font
@@
 		)
 		(property "Datasheet" "~"
-			(at 40.64 44.45 0)
+			(at 40.64 46.99 0)
 			(effects
 				(font
@@
 		)
 		(property "Description" "Generic screw terminal, single row, 01x02, script generated (kicad-library-utils/schlib/autogen/connector/)"
-			(at 40.64 44.45 0)
+			(at 40.64 46.99 0)
 			(effects
 				(font
@@
 	(symbol
 		(lib_id "Connector:Screw_Terminal_01x02")
-		(at 182.88 49.53 0)
-		(mirror x)
+		(at 182.88 46.99 0)
 		(unit 1)
 		(exclude_from_sim no)
@@
 		(dnp no)
 		(property "Reference" "J4"
-			(at 182.88 42.926 0)
+			(at 182.88 53.594 0)
 			(effects
 				(font
@@
 		)
 		(property "Value" "Motor"
-			(at 183.388 44.704 0)
+			(at 183.388 51.816 0)
 			(effects
 				(font
@@
 		)
 		(property "Footprint" "TerminalBlock_Phoenix:TerminalBlock_Phoenix_MKDS-1,5-2-5.08_1x02_P5.08mm_Horizontal"
-			(at 182.88 49.53 0)
+			(at 182.88 46.99 0)
 			(effects
 				(font
@@
 		)
 		(property "Datasheet" "~"
-			(at 182.88 49.53 0)
+			(at 182.88 46.99 0)
 			(effects
 				(font
@@
 		)
 		(property "Description" "Generic screw terminal, single row, 01x02, script generated (kicad-library-utils/schlib/autogen/connector/)"
-			(at 182.88 49.53 0)
-			(effects
-				(font
+			(at 182.88 46.99 0)
+			(effects
+				(font
