File: KiCad/proj_seients/proj_seients.kicad_pcb (KiCad board)
At the start: 2 copper layers, 126 x 89.4 mm, 102 parts, among them J1 BATERIA 12V, J10 Screw_Terminal_01x05, J11 FCarrera, J12 FCarrera, J13 FCarrera, J14 FCarrera, J17 FCarrera, J19 J_SENSOR_TEMP, J2 5f0857756ylz, J3 DE9_Pins, J4 Motor, J5 Motor, J6 Motor, J7 Manta_Asiento, J8 DE9_Socket, J9 FCarrera, Q1 IRLZ44N, SW1 SW_Push, SW2 SW_Push, SW3 SW_Push, SW4 SW_Push, SW5 SW_Push, SW6 SW_Push, SW7 SW_Push, U1 PIC24HJ128GP502, U10 MAX3232, U11 PCF8574AP, U2 LM2596S-5, U3 LM1117DT-3.3, U4 MCP2562-E-SN, U5 PCA9685BS, U6 DRV8871DDA, U7 DRV8871DDA, U8 DRV8871DDA, U9 24LC256, Y1 8MHz

Commit message: Versió 3.0
Parts:
- removed the REF** at (197.0, 68.2)
- removed the REF** at (197.1, 149.1)
- removed the REF** at (78.8, 149.0)
- removed the REF** at (79.0, 67.7)
- added R17: 10k, Resistor_SMD:R_0805_2012Metric, F.Cu at (220.5, 30.4)
- added R18: 10k, Resistor_SMD:R_0805_2012Metric, F.Cu at (220.5, 33.3)
- added R19: 10k, Resistor_SMD:R_0805_2012Metric, F.Cu at (220.5, 36.3)
- added R20: 10k, Resistor_SMD:R_0805_2012Metric, F.Cu at (220.5, 39.2)
- added R22: 10k, Resistor_SMD:R_0805_2012Metric, F.Cu at (220.5, 42.2)
- added R27: 10k, Resistor_SMD:R_0805_2012Metric, F.Cu at (220.5, 45.1)
- added REF**: MountingHole_3.2mm_M3, MountingHole:MountingHole_3.2mm_M3, F.Cu at (68.0, 147.8)
- added REF**: MountingHole_3.2mm_M3, MountingHole:MountingHole_3.2mm_M3, F.Cu at (217.5, 145.9)
- added REF**: MountingHole_3.2mm_M3, MountingHole:MountingHole_3.2mm_M3, F.Cu at (67.4, 68.8)
- added REF**: MountingHole_3.2mm_M3, MountingHole:MountingHole_3.2mm_M3, F.Cu at (220.2, 68.9)
- moved R25 188.8 mm to (267.6, 63.2), turned to 0 degrees
- moved C36 188.2 mm to (254.3, 59.2), turned to 0 degrees
- moved J14 167.1 mm to (277.2, 51.0), turned to 0 degrees
- moved J12 164.4 mm to (268.0, 51.0), turned to 0 degrees
- moved U11 163.2 mm to (273.2, 28.7), turned to 0 degrees
- moved J13 160.9 mm to (272.6, 51.0), turned to 0 degrees
- moved R24 155.6 mm to (267.6, 60.2), turned to 0 degrees
- moved R13 154.3 mm to (258.8, 66.1)
- moved C27 153.6 mm to (249.9, 59.2)
- moved C35 143.3 mm to (254.3, 56.2)
- moved SW2 137.2 mm to (230.2, 15.1), turned to 0 degrees
- moved C28 134.1 mm to (249.9, 62.2), turned to 0 degrees
- moved J11 133.0 mm to (263.4, 51.0), turned to 0 degrees
- moved C24 130.9 mm to (249.9, 50.2)
- moved R23 128.2 mm to (267.6, 57.3), turned to 0 degrees
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Routing:
- net 3.3V: track 414.3 -> 166.1 mm, vias 2 -> 0
- net 5V: track 177.1 -> 38.9 mm
- net Net-(J10-Pin_1): track 109.0 -> 23.9 mm, vias 4 -> 0
- net LIM_POS_MIN: track 73.5 -> 0.00 mm, vias 2 -> 0
- net LIM_AL_MIN: track 70.1 -> 0.00 mm, vias 1 -> 0
- net CALEFACCIÓ: track 78.7 -> 12.4 mm, vias 3 -> 0
- net Net-(U11-P1): track 52.7 -> 0.00 mm, vias 1 -> 0
- net LIM_REC_MAX: track 52.4 -> 0.00 mm, vias 1 -> 0
- net LIM_REC_MIN: track 51.8 -> 0.00 mm, vias 2 -> 0
- net 12V: track 136.5 -> 183.3 mm
- net LIM_AL_MAX: track 45.4 -> 0.00 mm, vias 3 -> 0
- net I2C_SCL: track 101.0 -> 58.9 mm, vias 3 -> 2
- net I2C_SDA: track 104.0 -> 62.2 mm, vias 6 -> 2
- net LIM_POS_MAX: track 40.1 -> 0.00 mm, vias 2 -> 0
- net Net-(U1-AVSS): track 46.5 -> 8.52 mm
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- removed copper zone on B.Cu, net GND
Other:
- board size 126 x 89.4 mm -> 160.8 x 87 mm
- board text removed: "Autors: Miguel Tovar i Pol Salas"
- board text removed: "Placa de Control - Seients Elèctrics"

Commit message: V3.2
Parts:
- moved J2 98.7 mm to (130.9, 49.8), turned to 180 degrees
- moved J19 96.1 mm to (149.8, 49.8), turned to 180 degrees
- moved J7 95.4 mm to (116.7, 49.8), turned to 180 degrees
- moved R3 94.0 mm to (139.2, 50.7), turned to -90 degrees
- moved R11 71.9 mm to (130.6, 59.9)
- moved Q1 71.9 mm to (135.9, 62.7)
- moved R10 60.4 mm to (135.9, 67.8), turned to -90 degrees
- moved D4 58.5 mm to (131.5, 68.8)
- moved J8 52.4 mm to (142.8, 137.6)
- moved J3 45.9 mm to (164.3, 137.5), turned to 0 degrees
- moved U4 38.1 mm to (155.1, 94.5)
- moved C7 38.1 mm to (145.9, 96.5)
- moved R1 38.1 mm to (131.0, 106.8)
- moved R5 38.1 mm to (138.7, 82.9)
- moved U10 38.1 mm to (163.3, 110.0)
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Connections:
- J1 pad 1: GND -> Net-(D1-A)
- J1 pad 2: Net-(D1-A) -> GND
- J7 pad 1: Net-(J7-Pin_1) -> 12V
- J7 pad 2: 12V -> Net-(J7-Pin_2)
- Q1 pad 2: Net-(J7-Pin_1) -> Net-(J7-Pin_2)
Routing:
- net 12V: track 183.3 -> 0.28 mm
- net Net-(J5-Pin_1): track 50.6 -> 3.03 mm, vias 2 -> 1
- net Net-(J6-Pin_1): track 47.3 -> 3.00 mm, vias 2 -> 1
- net Net-(J5-Pin_2): track 45.6 -> 2.66 mm, vias 2 -> 1
- net I2C_SCL: track 58.9 -> 16.6 mm
- net Net-(J4-Pin_1): track 43.3 -> 2.70 mm, vias 2 -> 1
- net Net-(J6-Pin_2): track 42.6 -> 3.02 mm, vias 2 -> 1
- net I2C_SDA: track 62.2 -> 23.4 mm
- net Net-(J4-Pin_2): track 40.5 -> 4.64 mm, vias 2 -> 1
- net 3.3V: track 166.1 -> 131.0 mm
- net Net-(J7-Pin_1): track 25.0 -> 0.00 mm
- net CAN_H: track 31.8 -> 9.20 mm
- net CAN_L: track 30.0 -> 8.90 mm
- net CINT: track 29.2 -> 12.9 mm
- net M2_IN1: track 22.8 -> 10.0 mm
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- added copper zone on F.Cu, net 12V
Other:
- board size 160.8 x 87 mm -> 130.7 x 109.7 mm

Commit message: V3.2
Parts:
- moved J6 0.83 mm to (76.9, 71.8)
- moved J4 0.83 mm to (76.9, 60.3)
- moved J5 0.83 mm to (76.9, 83.4)
Changed lines of the file:
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@@
 	(footprint "TerminalBlock_Phoenix:TerminalBlock_Phoenix_MKDS-1,5-2-5.08_1x02_P5.08mm_Horizontal"
 		(layer "F.Cu")
-		(at 76.8 84.22 -90)
+		(at 76.9 83.4 -90)
 		(descr "Terminal Block Phoenix MKDS-1,5-2-5.08, 2 pins, pitch 5.08mm, size 10.2x9.8mm, drill diameter 1.3mm, pad diameter 2.6mm, http://www.farnell.com/datasheets/100425.pdf, script-generated using https://gitlab.com/kicad/libraries/kicad-footprint-generator/-/tree/master/scripts/TerminalBlock_Phoenix")
 		(tags "THT Terminal Block Phoenix MKDS-1,5-2-5.08 pitch 5.08mm size 10.2x9.8mm drill 1.3mm pad 2.6mm")
@@
 	(footprint "TerminalBlock_Phoenix:TerminalBlock_Phoenix_MKDS-1,5-2-5.08_1x02_P5.08mm_Horizontal"
 		(layer "F.Cu")
-		(at 76.8 72.62 -90)
+		(at 76.9 71.8 -90)
 		(descr "Terminal Block Phoenix MKDS-1,5-2-5.08, 2 pins, pitch 5.08mm, size 10.2x9.8mm, drill diameter 1.3mm, pad diameter 2.6mm, http://www.farnell.com/datasheets/100425.pdf, script-generated using https://gitlab.com/kicad/libraries/kicad-footprint-generator/-/tree/master/scripts/TerminalBlock_Phoenix")
 		(tags "THT Terminal Block Phoenix MKDS-1,5-2-5.08 pitch 5.08mm size 10.2x9.8mm drill 1.3mm pad 2.6mm")
@@
 	(footprint "TerminalBlock_Phoenix:TerminalBlock_Phoenix_MKDS-1,5-2-5.08_1x02_P5.08mm_Horizontal"
 		(layer "F.Cu")
-		(at 76.8 61.12 -90)
+		(at 76.9 60.3 -90)
 		(descr "Terminal Block Phoenix MKDS-1,5-2-5.08, 2 pins, pitch 5.08mm, size 10.2x9.8mm, drill diameter 1.3mm, pad diameter 2.6mm, http://www.farnell.com/datasheets/100425.pdf, script-generated using https://gitlab.com/kicad/libraries/kicad-footprint-generator/-/tree/master/scripts/TerminalBlock_Phoenix")
 		(tags "THT Terminal Block Phoenix MKDS-1,5-2-5.08 pitch 5.08mm size 10.2x9.8mm drill 1.3mm pad 2.6mm")

Commit message: V3.3
Parts:
- moved U11 171.5 mm to (128.6, 120.9), turned to 90 degrees
- moved R18 148.9 mm to (133.8, 138.2), turned to 90 degrees
- moved SW3 143.4 mm to (153.5, 144.8), turned to 90 degrees
- moved R17 142.2 mm to (148.6, 137.4), turned to 90 degrees
- moved SW2 141.0 mm to (153.6, 133.4), turned to 90 degrees
- moved SW5 138.5 mm to (138.8, 144.8), turned to 90 degrees
- moved SW7 137.6 mm to (124.2, 145.6), turned to 90 degrees
- moved SW4 136.4 mm to (138.9, 133.5), turned to 90 degrees
- moved SW6 135.6 mm to (124.0, 133.7), turned to 90 degrees
- moved R27 132.3 mm to (133.7, 128.0), turned to -90 degrees
- moved R20 127.2 mm to (148.6, 128.0), turned to -90 degrees
- moved R22 124.5 mm to (163.2, 137.3), turned to 90 degrees
- moved J17 124.1 mm to (157.7, 49.0), turned to 180 degrees
- moved R19 121.4 mm to (163.2, 127.9), turned to -90 degrees
- moved J14 114.9 mm to (162.3, 49.0), turned to 180 degrees
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Routing:
- net 3.3V: track 131.0 -> 12.1 mm
- net TX: track 5.22 -> 0.00 mm
- net CAN_H: track 9.20 -> 4.06 mm
- net CAN_L: track 8.90 -> 4.07 mm
- net RX: track 4.62 -> 0.00 mm
- net GND: vias 23 -> 24

Commit message: V3.4
Parts:
- moved C18 115.6 mm to (133.8, 143.8), turned to 90 degrees
- moved C24 111.6 mm to (148.6, 141.4), turned to 90 degrees
- moved C36 110.0 mm to (124.6, 113.5), turned to 90 degrees
- moved R25 95.0 mm to (147.4, 102.1)
- moved C19 93.3 mm to (163.2, 141.7), turned to 90 degrees
- moved R26 93.2 mm to (147.4, 100.0)
- moved R16 92.8 mm to (147.4, 106.8)
- moved C21 86.8 mm to (147.1, 125.0)
- moved C22 80.0 mm to (142.8, 109.6)
- moved C20 75.9 mm to (164.2, 123.8), turned to 180 degrees
- moved R14 73.4 mm to (158.2, 54.4)
- moved R15 69.2 mm to (162.8, 54.4)
- moved R23 63.9 mm to (172.2, 54.4)
- moved R13 61.4 mm to (167.5, 54.4)
- moved R24 59.9 mm to (176.6, 54.4)
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Connections:
- U6 pad 6: Net-(J6-Pin_2) -> Net-(J6-Pin_1)
- U6 pad 8: Net-(J6-Pin_1) -> Net-(J6-Pin_2)
- U7 pad 6: Net-(J4-Pin_2) -> Net-(J4-Pin_1)
- U7 pad 8: Net-(J4-Pin_1) -> Net-(J4-Pin_2)
- U8 pad 6: Net-(J5-Pin_2) -> Net-(J5-Pin_1)
- U8 pad 8: Net-(J5-Pin_1) -> Net-(J5-Pin_2)
Routing:
- net Net-(J7-Pin_2): track 0.00 -> 37.0 mm
- net Net-(U11-P2): track 0.00 -> 34.1 mm
- net Net-(J4-Pin_2): track 4.64 -> 34.7 mm, vias 1 -> 0
- net Net-(J5-Pin_2): track 2.66 -> 31.3 mm, vias 1 -> 0
- net Net-(J6-Pin_2): track 3.02 -> 31.1 mm, vias 1 -> 0
- net Net-(J5-Pin_1): track 3.03 -> 30.2 mm, vias 1 -> 0
- net Net-(J4-Pin_1): track 2.70 -> 29.8 mm, vias 1 -> 0
- net INT_BOTONERA: track 0.00 -> 25.2 mm
- net Net-(J6-Pin_1): track 3.00 -> 26.6 mm, vias 1 -> 0
- net RX: track 0.00 -> 23.1 mm
- net CAN_H: track 4.06 -> 26.0 mm
- net TX: track 0.00 -> 20.7 mm
- net CAN_L: track 4.07 -> 23.0 mm
- net M3_IN2: track 5.65 -> 21.5 mm, vias 0 -> 2
- net M3_IN1: track 7.34 -> 23.1 mm, vias 0 -> 2
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- added copper zone on F.Cu, net 3.3V
- added copper zone on B.Cu, net GND

Commit message: V3.5
Parts:
- moved C4 32.8 mm to (104.3, 109.9), turned to -90 degrees
- moved U3 31.5 mm to (113.4, 113.9), turned to 0 degrees
- moved C18 14.8 mm to (148.6, 143.2)
- moved SW7 14.8 mm to (138.9, 145.0)
- moved R18 14.8 mm to (148.6, 137.7)
- moved C24 14.8 mm to (133.8, 141.6)
- moved R17 14.8 mm to (133.8, 137.6)
- moved SW5 14.8 mm to (124.1, 145.0)
- moved C36 7.61 mm to (124.3, 121.0)
- moved D2 6.53 mm to (91.3, 110.6)
- moved D1 3.98 mm to (103.8, 128.8)
- moved R1 1.67 mm to (132.5, 107.6), turned to 180 degrees
- moved C21 0.10 mm to (147.1, 124.9)
Routing:
- net GND: track 3.60 -> 219.5 mm, vias 26 -> 110
- net LIM_AL_MIN: track 0.00 -> 85.4 mm, vias 0 -> 2
- net 5V: track 33.3 -> 106.2 mm, vias 0 -> 2
- net LIM_REC_MAX: track 0.00 -> 71.2 mm, vias 0 -> 2
- net LIM_AL_MAX: track 0.00 -> 68.8 mm, vias 0 -> 2
- net I2C_SCL: track 28.4 -> 96.2 mm, vias 0 -> 3
- net I2C_SDA: track 32.6 -> 99.1 mm, vias 0 -> 3
- net LIM_REC_MIN: track 0.00 -> 62.3 mm
- net CINT: track 6.17 -> 64.4 mm, vias 1 -> 2
- net LIM_POS_MIN: track 9.37 -> 61.0 mm, vias 0 -> 2
- net TEMP_SEIENT: track 5.55 -> 53.4 mm, vias 0 -> 1
- net LIM_POS_MAX: track 9.37 -> 55.8 mm, vias 0 -> 2
- net UART_RX: track 0.00 -> 44.7 mm, vias 0 -> 2
- net UART_TX: track 0.00 -> 42.8 mm, vias 0 -> 2
- net Net-(U11-P4): track 14.2 -> 44.0 mm, vias 0 -> 1
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
Commit message: V3.6
Changed lines of the file:
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@@
-	)
-	(segment
-		(start 142.2 102.8)
-		(end 140.56 102.8)
-		(width 0.25)
-		(layer "F.Cu")
-		(net 24)
 	)
 	(segment
@@
 	)
 	(segment
-		(start 140.56 102.8)
-		(end 140.5 102.74)
+		(start 143.9 102.8)
+		(end 140.56 102.8)
 		(width 0.25)
 		(layer "F.Cu")
@@
 	)
 	(segment
+		(start 140.56 102.8)
+		(end 140.5 102.74)
+		(width 0.25)
+		(layer "F.Cu")
+		(net 24)
+	)
+	(segment
 		(start 171.275 54.4)
 		(end 171.275 50.835)
@@
 	)
 	(via
-		(at 142.2 102.8)
+		(at 143.9 102.8)
 		(size 0.6)
 		(drill 0.3)
@@
 	)
 	(segment
-		(start 170 58.9)
+		(start 144.5 102.8)
 		(end 170 77.3)
 		(width 0.25)
@@
 	(segment
 		(start 170 77.3)
-		(end 144.5 102.8)
+		(end 170 58.9)
 		(width 0.25)
 		(layer "B.Cu")
@@
 	)
 	(segment
-		(start 144.5 102.8)
-		(end 144.3 102.8)
+		(start 143.9 102.8)
+		(end 144.5 102.8)
 		(width 0.25)
 		(layer "B.Cu")
-		(net 24)
-	)
-	(segment
-		(start 144.3 102.8)
-		(end 142.2 102.8)
-		(width 0.25)
-		(layer "B.Cu")
