File: KiCad/proj_seients/proj_seients.kicad_pcb (KiCad board)
At the start: 2 copper layers, 130.7 x 109.7 mm, 108 parts, among them J1 BATERIA 12V, J10 Screw_Terminal_01x05, J11 FCarrera, J12 FCarrera, J13 FCarrera, J14 FCarrera, J17 FCarrera, J19 J_SENSOR_TEMP, J2 5f0857756ylz, J3 DE9_Pins, J4 Motor, J5 Motor, J6 Motor, J7 Manta_Asiento, J8 DE9_Socket, J9 FCarrera, Q1 IRLZ44N, SW1 SW_Push, SW2 SW_Push, SW3 SW_Push, SW4 SW_Push, SW5 SW_Push, SW6 SW_Push, SW7 SW_Push, U1 PIC24HJ128GP502, U10 MAX3232, U11 PCF8574AP, U2 LM2596S-5, U3 LM1117DT-3.3, U4 MCP2562-E-SN, U5 PCA9685BS, U6 DRV8871DDA, U7 DRV8871DDA, U8 DRV8871DDA, U9 24LC256, Y1 8MHz

Commit message: Fix alguns errors en millora-pcb
Routing:
- net 5V: track 106.2 -> 104.9 mm
Changed lines of the file:
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@@
-	)
-	(segment
-		(start 105.4 118.9)
-		(end 105.7 118.9)
-		(width 1)
-		(layer "F.Cu")
-		(net 3)
 	)
 	(segment
@@
 	)
 	(segment
-		(start 105.7 118.9)
-		(end 108.4 116.2)
+		(start 108.5 118.9)
+		(end 118 118.9)
 		(width 1)
 		(layer "F.Cu")
@@
 	(segment
 		(start 105.4 118.9)
-		(end 118 118.9)
-		(width 1)
+		(end 108.5 118.9)
+		(width 1)
+		(layer "F.Cu")
+		(net 3)
+	)
+	(segment
+		(start 108.4 116.2)
+		(end 108.4 118.8)
+		(width 0.5)
 		(layer "F.Cu")
 		(net 3)
@@
 		(end 118.9 116.6)
 		(width 1)
+		(layer "F.Cu")
+		(net 3)
+	)
+	(segment
+		(start 108.4 118.8)
+		(end 108.5 118.9)
+		(width 0.5)
 		(layer "F.Cu")
 		(net 3)
@@
 	)
 	(segment
-		(start 131.2 95.12)
-		(end 136.2 95.12)
-		(width 0.25)
-		(layer "F.Cu")
-		(net 25)
-	)
-	(segment
-		(start 136.2 95.12)
-		(end 138.5 92.82)
-		(width 0.25)
-		(layer "F.Cu")
-		(net 25)
-	)
-	(segment
 		(start 142.8 88)
 		(end 142.8 87.5)
@@
 	)
 	(segment
-		(start 140.067678 97.66)
-		(end 140.5 97.66)
+		(start 139.475001 97.66)
+		(end 138.5 96.684999)
 		(width 0.25)
 		(layer "F.Cu")
@@
 	)
 	(segment
-		(start 138.5 92.82)
-		(end 138.5 90.5)
+		(start 138.5 95)
+		(end 138.5 94.5)
+		(width 0.25)
+		(layer "F.Cu")
+		(net 25)
+	)
+	(segment
+		(start 131.2 95.12)
+		(end 137.88 95.12)
 		(width 0.25)
 		(layer "F.Cu")
@@
 	)
 	(segment
+		(start 138.5 94.5)
+		(end 138.5 90.5)
+		(width 0.25)
+		(layer "F.Cu")
+		(net 25)
+	)
+	(segment
 		(start 142.8 87.5)
 		(end 144.3 87.5)
@@
 	)
 	(segment
+		(start 138.5 96.684999)
+		(end 138.5 95)
+		(width 0.25)
+		(layer "F.Cu")
+		(net 25)
+	)
+	(segment
 		(start 144.3 87.5)
 		(end 148.8 87.5)
@@
 	)
 	(segment
-		(start 137.527678 95.12)
-		(end 140.067678 97.66)
+		(start 140.5 97.66)
+		(end 139.475001 97.66)
 		(width 0.25)
 		(layer "F.Cu")
@@
 	)
 	(segment
-		(start 136.2 95.12)
-		(end 137.527678 95.12)
+		(start 137.88 95.12)
+		(end 138.5 94.5)
 		(width 0.25)
 		(layer "F.Cu")
@@
 	(segment
 		(start 138.7 106.8)
-		(end 140.4 106.8)
+		(end 140 106.8)
 		(width 0.25)
 		(layer "F.Cu")
@@
 	)
 	(segment
+		(start 140 106.4)
+		(end 140 106.8)
+		(width 0.25)
+		(layer "F.Cu")
+		(net 64)
+	)
+	(segment
 		(start 139.7 106.1)
-		(end 140.4 106.8)
+		(end 140 106.4)
 		(width 0.25)
 		(layer "F.Cu")
@@
 		(width 0.25)
 		(layer "F.Cu")
+		(net 64)
+	)
+	(segment
+		(start 140 106.8)
+		(end 140.4 106.8)
+		(width 0.25)
+		(layer "F.Cu")

Commit message: V3.6
Parts:
- removed C33, C34: 100nF, Capacitor_SMD:C_0805_2012Metric
- added 12V: TestPoint_Pad_D1.0mm, TestPoint:TestPoint_Pad_D1.0mm, F.Cu at (67.0, 134.2)
- added 3,3V: TestPoint_Pad_D1.0mm, TestPoint:TestPoint_Pad_D1.0mm, F.Cu at (108.5, 148.5)
- added 5V: TestPoint_Pad_D1.0mm, TestPoint:TestPoint_Pad_D1.0mm, F.Cu at (102.8, 140.5)
- added GND: TestPoint_Pad_D1.0mm, TestPoint:TestPoint_Pad_D1.0mm, F.Cu at (151.6, 101.8)
- added GND: TestPoint_Pad_D1.0mm, TestPoint:TestPoint_Pad_D1.0mm, F.Cu at (104.2, 147.2)
- added GND: TestPoint_Pad_D1.0mm, TestPoint:TestPoint_Pad_D1.0mm, F.Cu at (67.0, 137.0)
- added I2C_SCL: TestPoint_Pad_D1.0mm, TestPoint:TestPoint_Pad_D1.0mm, F.Cu at (144.8, 104.0)
- added I2C_SDA: TestPoint_Pad_D1.0mm, TestPoint:TestPoint_Pad_D1.0mm, F.Cu at (151.5, 97.8)
- moved J3 77.6 mm to (114.0, 138.2), turned to 0 degrees
- moved R2 59.3 mm to (117.2, 134.0), turned to 0 degrees
- moved J1 52.1 mm to (72.0, 110.3), turned to -90 degrees
- moved U4 50.1 mm to (116.3, 126.2), turned to 180 degrees
- moved J17 33.9 mm to (176.0, 81.2), turned to -90 degrees
- moved D2 32.9 mm to (89.2, 143.4)
- moved D3 31.6 mm to (86.0, 124.4)
- moved D1 31.3 mm to (73.4, 136.4), turned to 90 degrees
- moved R12 31.0 mm to (82.1, 124.4)
- moved C2 30.5 mm to (108.2, 134.9), turned to 90 degrees
- moved R21 29.4 mm to (169.3, 81.2), turned to -90 degrees
- moved C1 29.0 mm to (83.5, 135.9), turned to 90 degrees
- moved J14 29.0 mm to (176.0, 76.6), turned to -90 degrees
- moved C23 27.8 mm to (164.7, 81.2), turned to 90 degrees
- moved J13 24.7 mm to (176.0, 72.0), turned to -90 degrees
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Connections:
- J1 pad 1: Net-(D1-A) -> GND
- J1 pad 2: GND -> Net-(D1-A)
- U1 pad 19: Net-(U1-AVSS) -> GND
- U1 pad 27: Net-(U1-AVSS) -> GND
- U1 pad 8: Net-(U1-AVSS) -> GND
Routing:
- net 5V: track 104.9 -> 0.00 mm, vias 2 -> 0
- net CAN_RX: track 12.1 -> 47.9 mm
- net GND: track 219.5 -> 253.1 mm, vias 110 -> 120
- net CAN_TX: track 12.1 -> 44.6 mm
- net Net-(U1-AVSS): track 30.5 -> 0.00 mm, vias 2 -> 0
- net Net-(J4-Pin_2): track 34.7 -> 11.2 mm
- net LIM_REC_MIN: track 62.3 -> 40.0 mm
- net Net-(J5-Pin_2): track 31.3 -> 9.38 mm
- net Net-(J6-Pin_2): track 31.1 -> 9.57 mm
- net Net-(J5-Pin_1): track 30.2 -> 10.2 mm
- net Net-(J4-Pin_1): track 29.8 -> 10.9 mm
- net LIM_REC_MAX: track 71.2 -> 53.5 mm
- net Net-(J6-Pin_1): track 26.6 -> 9.43 mm
- net Net-(U11-P5): track 45.1 -> 30.8 mm
- net TX: track 20.7 -> 8.28 mm
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- added copper zone on F.Cu, net 5V
Other:
- board size 130.7 x 109.7 mm -> 117.7 x 109.7 mm

Commit message: V3.7
Parts:
- moved C25 41.0 mm to (125.4, 132.6), turned to -90 degrees
- moved C26 34.4 mm to (125.4, 127.6), turned to 90 degrees
- moved J19 26.5 mm to (119.3, 50.0)
- moved R3 26.5 mm to (110.0, 50.9)
- moved J7 15.0 mm to (131.7, 49.9)
- moved J2 14.7 mm to (145.6, 49.7)
- moved R17 2.66 mm to (142.6, 138.5)
- moved SW5 2.66 mm to (132.9, 145.9)
- moved C24 2.66 mm to (142.6, 142.6)
- moved R27 2.66 mm to (142.5, 129.0)
- moved SW6 2.66 mm to (132.8, 134.6)
- moved I2C_SCL 2.46 mm to (147.2, 104.6)
- moved D4 1.99 mm to (133.1, 70.0)
- moved REF** 0.98 mm to (67.8, 46.6)
- moved REF** 0.40 mm to (176.7, 46.4)
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Connections:
- net Net-(D2-K) renamed /potencia/SW_5V
- net Net-(D3-A) renamed /potencia/NET_LED_BAT
- net Net-(D4-A) renamed /potencia/NET_LED_CAL
- net Net-(J4-Pin_1) renamed /potencia/M1_OUT_A
- net Net-(J4-Pin_2) renamed /potencia/M1_OUT_B
- net Net-(J5-Pin_1) renamed /potencia/M2_OUT_A
- net Net-(J5-Pin_2) renamed /potencia/M2_OUT_B
- net Net-(J6-Pin_1) renamed /potencia/M3_OUT_A
- net Net-(J6-Pin_2) renamed /potencia/M3_OUT_B
- net Net-(J7-Pin_2) renamed /potencia/OUT_CALEFACCIO
- net Net-(U6-ILIM) renamed /potencia/ILIM_3
- net Net-(U7-ILIM) renamed /potencia/ILIM_1
- net Net-(U8-ILIM) renamed /potencia/ILIM_2
Routing:
- net /potencia/OUT_CALEFACCIO: track 38.2 -> 22.8 mm, vias 1 -> 0
- net CINT: track 64.4 -> 73.4 mm
- net LIM_AL_MAX: track 56.8 -> 64.1 mm, vias 2 -> 0
- net Net-(U11-P5): track 30.8 -> 35.4 mm, vias 1 -> 0
- net Net-(U11-P0): track 38.0 -> 33.6 mm
- net TEMP_SEIENT: track 54.3 -> 57.2 mm, vias 1 -> 0
- net LIM_REC_MIN: track 40.0 -> 37.4 mm, vias 0 -> 2
- net LIM_AL_MIN: track 79.8 -> 78.2 mm
- net LIM_POS_MIN: track 62.7 -> 61.2 mm, vias 2 -> 0
- net M3_IN1: track 13.9 -> 15.0 mm, vias 2 -> 0
- net /potencia/NET_LED_CAL: track 3.55 -> 2.41 mm
- net I2C_SCL: track 98.3 -> 99.4 mm
- net M1_IN2: track 30.2 -> 31.0 mm, vias 2 -> 0
- net M3_IN2: track 13.5 -> 14.3 mm, vias 2 -> 0
- net M2_IN1: track 20.5 -> 20.9 mm, vias 2 -> 0
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
Commit message: V3.8
Parts:
- moved D1 35.0 mm to (98.9, 112.3), turned to 180 degrees
- moved 12V 24.1 mm to (83.5, 116.8)
- moved GND 24.1 mm to (83.5, 119.5)
- moved C22 22.3 mm to (147.9, 131.4), turned to 180 degrees
- moved C35 19.2 mm to (165.2, 57.5)
- moved J17 19.2 mm to (176.5, 62.0)
- moved R24 19.2 mm to (169.7, 57.4)
- moved C23 19.2 mm to (165.2, 62.1)
- moved J14 19.2 mm to (176.5, 57.4)
- moved R21 19.2 mm to (169.8, 62.0)
- moved J1 17.4 mm to (85.7, 99.7)
- moved C21 17.1 mm to (174.3, 130.7), turned to 180 degrees
- moved SW4 16.8 mm to (166.5, 134.7)
- moved REF** 15.5 mm to (83.0, 147.9)
- moved REF** 15.2 mm to (83.0, 46.3)
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Connections:
- net /potencia/ILIM_1 renamed Net-(U7-ILIM)
- net /potencia/ILIM_2 renamed Net-(U8-ILIM)
- net /potencia/ILIM_3 renamed Net-(U6-ILIM)
- net /potencia/M1_OUT_A renamed Net-(J4-Pin_1)
- net /potencia/M1_OUT_B renamed Net-(J4-Pin_2)
- net /potencia/M2_OUT_A renamed Net-(J5-Pin_1)
- net /potencia/M2_OUT_B renamed Net-(J5-Pin_2)
- net /potencia/M3_OUT_A renamed Net-(J6-Pin_1)
- net /potencia/M3_OUT_B renamed Net-(J6-Pin_2)
- net /potencia/NET_LED_BAT renamed Net-(D3-A)
- net /potencia/NET_LED_CAL renamed Net-(D4-A)
- net /potencia/OUT_CALEFACCIO renamed Net-(J7-Pin_2)
- net /potencia/SW_5V renamed Net-(D2-K)
- U1 pad 26: CALEFACCIÓ -> LIM_REC_MAX
- U1 pad 3: LIM_REC_MAX -> CALEFACCIÓ
Routing:
- net LIM_REC_MIN: track 37.4 -> 58.9 mm, vias 2 -> 0
- net Net-(U11-P2): track 45.3 -> 32.6 mm
- net I2C_SCL: track 99.4 -> 111.1 mm, vias 1 -> 0
- net GND: track 253.1 -> 243.8 mm, vias 120 -> 119
- net LIM_POS_MAX: track 64.0 -> 54.8 mm
- net CINT: track 73.4 -> 64.1 mm, vias 2 -> 0
- net LIM_POS_MIN: track 61.2 -> 52.0 mm
- net Net-(U11-P4): track 55.3 -> 64.0 mm, vias 1 -> 0
- net LIM_REC_MAX: track 53.8 -> 62.5 mm, vias 2 -> 0
- net I2C_SDA: track 105.9 -> 114.5 mm, vias 1 -> 0
- net LIM_AL_MAX: track 64.1 -> 55.5 mm
- net LIM_AL_MIN: track 78.2 -> 70.6 mm
- net Net-(U11-P3): track 35.6 -> 42.2 mm, vias 2 -> 0
- net Net-(J10-Pin_1): track 23.9 -> 18.0 mm
- net Net-(D2-K): track 14.0 -> 17.0 mm
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Other:
- board size 117.7 x 109.7 mm -> 101.8 x 109.7 mm

Commit message: V3.8
Parts:
- moved D3 1.41 mm to (87.4, 124.7)
- moved R12 1.41 mm to (83.5, 124.7)
- moved D4 1.38 mm to (132.9, 68.6)
- moved C4 1.18 mm to (116.9, 125.4)
- moved U3 1.18 mm to (118.1, 116.6)
- moved C36 1.12 mm to (129.7, 109.2)
- moved D2 0.91 mm to (98.0, 141.6)
Routing:
- net LIM_AL_MAX: track 55.5 -> 57.3 mm
- net GND: track 243.8 -> 242.2 mm
- net Net-(D2-K): track 17.0 -> 15.5 mm
- net I2C_SDA: track 114.5 -> 113.1 mm
- net I2C_SCL: track 111.1 -> 109.7 mm
- net LIM_AL_MIN: track 70.6 -> 71.5 mm
- net Net-(U11-P0): track 35.5 -> 36.1 mm
- net Net-(U11-P4): track 64.0 -> 63.4 mm
- net M3_IN1: track 15.0 -> 14.5 mm
- net UART_TX: track 38.7 -> 39.3 mm
- net CAN_RX: track 48.0 -> 48.5 mm
